File: pcb/noria.sch (KiCad schematic (older format))
At the start: 61 parts, among them J1 AudioJack4, J2 USB_C_Receptacle_USB2.0, SW1 SW_PUSH, SW10 SW_PUSH, SW11 SW_PUSH, SW12 SW_PUSH, SW13 SW_PUSH, SW14 SW_PUSH, SW15 SW_PUSH, SW16 SW_PUSH, SW17 SW_PUSH, SW18 SW_PUSH, SW19 SW_PUSH, SW2 SW_PUSH, SW20 SW_PUSH, SW21 SW_PUSH, SW22 SW_PUSH, SW23 SW_PUSH, SW24 SW_PUSH, SW25 SW_PUSH, SW3 SW_PUSH, SW4 SW_PUSH, SW5 SW_PUSH, SW6 SW_PUSH, SW7 SW_PUSH, SW8 SW_PUSH, SW9 SW_PUSH, U1 holyiot18010, U2 M25PX32-VMW

Commit message: Finished iteration 1
Parts:
- removed D1, D10, D11, D12, D13, D14, D15, D16, D17, D18, D19, D2, D20, D21, D22, D23, D24, D25, D3, D4, D5, D6, D7, D8, D9: D, Diode_SMD:D_SOD-323_HandSoldering, symbol Device:D
- removed J1: AudioJack4, Connector_Audio:Jack_3.5mm_CUI_SJ-3524-SMT_Horizontal, symbol Connector:AudioJack4
- removed SW1, SW10, SW11, SW12, SW13, SW14, SW15, SW16, SW17, SW18, SW19, SW2, SW20, SW21, SW22, SW23, SW24, SW25, SW3, SW4, SW5, SW6, SW7, SW8, SW9: SW_PUSH, kicad-footprints:CherryMX_Choc_Hotswap, symbol kbd:SW_PUSH
- removed U2: M25PX32-VMW, Package_SO:SOIJ-8_5.3x5.3mm_P1.27mm, symbol Memory_Flash:M25PX32-VMW
- added C3, C4: 1u, lib:C_0603_1608Metric_Pad1.08x0.95mm_HandSolder_mirror, symbol Device:C
- added H1, H2: MountingHole, kicad-footprints:spacer_m2, symbol Mechanical:MountingHole
- added H3, H4, H5, H6, H7: MountingHole, MountingHole:MountingHole_3.5mm_Pad_Via, symbol Mechanical:MountingHole_Pad
- added H8, H9: MountingHole, kicad-footprints:M2_Hole_TH, symbol Mechanical:MountingHole
- added J10, J9: MJ-4PP-9, kicad-footprints:MJ-4PP-9_1side, symbol kbd:MJ-4PP-9
- added J2: USB_C_Receptacle_USB2.0, Connector_USB:USB_C_Receptacle_HRO_TYPE-C-31-M-12, symbol Connector:USB_C_Receptacle_USB2.0
- added J4: SWD, Connector_PinHeader_2.54mm:PinHeader_1x04_P2.54mm_Horizontal, symbol Connector_Generic:Conn_01x04
- added J7: display, Connector_PinHeader_2.54mm:PinHeader_1x04_P2.54mm_Vertical, symbol Connector_Generic:Conn_01x04
- added J8: Conn_01x03, Connector_PinHeader_2.54mm:PinHeader_1x03_P2.54mm_Vertical, symbol Connector_Generic:Conn_01x03
- added JP1, JP11, JP12, JP2: SolderJumper_3_Bridged12, Jumper:SolderJumper-3_P1.3mm_Bridged12_Pad1.0x1.5mm, symbol Jumper:SolderJumper_3_Bridged12
- added JP10, JP3, JP4, JP5, JP6, JP7, JP8, JP9: SolderJumper_2_Open, kicad-footprints:Jumper, symbol Jumper:SolderJumper_2_Open
- added R1, R2: 4.7K, lib:R_0603_1608Metric_Pad0.98x0.95mm_HandSolder, symbol Device:R
- added R11, R9: 22, Resistor_SMD:R_0603_1608Metric_Pad0.98x0.95mm_HandSolder, symbol Device:R
- added U1, U4: MX25R3235FM1xx0, Package_SO:SOP-8_3.9x4.9mm_P1.27mm, symbol Memory_Flash:MX25R3235FM1xx0
- added U3: holyiot18010, lib:holyiot18010_no_inner, symbol lib:holyiot18010_no_pads
- added U5, U6: TLV73333PDBV, Package_TO_SOT_SMD:SOT-23-5, symbol Regulator_Linear:TLV73333PDBV
- C1: renamed from C2; value C -> 100n; footprint Capacitor_SMD:C_0805_2012Metric_Pad1.18x1.45mm_HandSolder -> Capacitor_SMD:C_0603_1608Metric_Pad1.08x0.95mm_HandSolder
- C2: renamed from C1; value C -> 100n; footprint Capacitor_SMD:C_0805_2012Metric_Pad1.18x1.45mm_HandSolder -> Capacitor_SMD:C_0603_1608Metric_Pad1.08x0.95mm_HandSolder
- R10: renamed from R2; value R -> 22
- R3: renamed from R1; value R -> 5.1K; footprint Resistor_SMD:R_0603_1608Metric_Pad0.98x0.95mm_HandSolder -> lib:R_0603_1608Metric_Pad0.98x0.95mm_HandSolder
- R4: value R -> 5.1K; footprint Resistor_SMD:R_0603_1608Metric_Pad0.98x0.95mm_HandSolder -> lib:R_0603_1608Metric_Pad0.98x0.95mm_HandSolder
- RSW1: footprint kicad-footprints:CherryMX_Choc_Hotswap -> kicad-footprints:ResetSW
- U2: renamed from U1; footprint lib:holyiot18010_mirror -> lib:holyiot18010_no_inner; symbol lib:holyiot18010 -> lib:holyiot18010_no_pads
- renumbered J2 to J3, R3 to R12
Connections:
- net labels added: CC1, CC2, QDEC_A, QDEC_B, SCLK_B, SCLK_T, SCL_B, SCL_T, SDA_B, SDA_T, SIO0_B, SIO0_T, SIO1_B, SIO1_T, SIO2_B, SIO2_T, SIO3_B, SIO3_T, SWCLK, UART0_RX, UART0_TX, USBB+, USBB-, USBC_+, USBC_-, USBT+, USBT-, nCS_B, nCS_T, nReset
- net labels removed: SWDCLK, USB+, USB-
- wire segments 102 -> 135
- no-connect marks 0 -> 4
Other:
- moved on the sheet: C1, C2, J3, R10, R12, R3, RSW1

Commit message: Update to latest design
Parts:
- removed J4: SWD, Connector_PinHeader_2.54mm:PinHeader_1x04_P2.54mm_Horizontal, symbol Connector_Generic:Conn_01x04
- added J1, J4: Conn_02x05_Odd_Even, Connector_PinHeader_1.27mm:PinHeader_2x05_P1.27mm_Vertical_SMD, symbol Connector_Generic:Conn_02x05_Odd_Even
- C1, C2: LCSC (none) -> C66501
- C3, C4: LCSC (none) -> C59782
- J10, J9: LCSC (none) -> C136687
- J2, J3: LCSC (none) -> C165948
- J7: LCSC (none) -> C2718488
- R1, R2: LCSC (none) -> C23162
- R10, R11, R12, R9: LCSC (none) -> C23345
- R3, R4: LCSC (none) -> C23186
- RSW1: LCSC (none) -> C498307
- U1, U4: value MX25R3235FM1xx0 -> BY25Q32BSTIG(T); LCSC (none) -> C394868
- U5, U6: LCSC (none) -> C134139
Connections:
- wire segments 135 -> 138
- no-connect marks 4 -> 12
