File: pcb/noria.kicad_pcb (KiCad board)
At the start: 2 copper layers, 160.8 x 113.7 mm, 61 parts, among them J1 AudioJack4, J2 USB_C_Receptacle_USB2.0, SW1 SW_PUSH, SW10 SW_PUSH, SW11 SW_PUSH, SW12 SW_PUSH, SW13 SW_PUSH, SW14 SW_PUSH, SW15 SW_PUSH, SW16 SW_PUSH, SW17 SW_PUSH, SW18 SW_PUSH, SW19 SW_PUSH, SW2 SW_PUSH, SW20 SW_PUSH, SW21 SW_PUSH, SW22 SW_PUSH, SW23 SW_PUSH, SW24 SW_PUSH, SW25 SW_PUSH, SW3 SW_PUSH, SW4 SW_PUSH, SW5 SW_PUSH, SW6 SW_PUSH, SW7 SW_PUSH, SW8 SW_PUSH, SW9 SW_PUSH, U1 holyiot18010, U2 M25PX32-VMW

Commit message: Finished iteration 1
Parts:
- removed the D14 at (-56.2, 145.4)
- removed the D25 at (-91.6, 142.5)
- removed J1: AudioJack4, Connector_Audio:Jack_3.5mm_CUI_SJ-3524-SMT_Horizontal
- removed the SW2 at (120.8, 78.5)
- removed the SW25 at (101.2, 108.6)
- removed the SW3 at (120.8, 97.6)
- removed the SW5 at (139.9, 57.0)
- removed the SW8 at (93.7, 138.1)
- added C3: 1u, lib:C_0603_1608Metric_Pad1.08x0.95mm_HandSolder_mirror, F.Cu at (106.0, 64.4)
- added C4: 1u, lib:C_0603_1608Metric_Pad1.08x0.95mm_HandSolder_mirror, F.Cu at (110.6, 60.4)
- added D13: D, lib:D3_SMD_v2_mirror, F.Cu at (129.4, 94.6)
- added D24: D, lib:D3_SMD_v2_mirror, F.Cu at (160.2, 111.7)
- added H1: MountingHole, kicad-footprints:spacer_m2, F.Cu at (206.6, 97.1)
- added H10: MountingHole, keyswitches:Stabilizer_MX_2u, F.Cu at (87.0, 131.4)
- added H11: MountingHole, keyswitches:Stabilizer_MX_2u, F.Cu at (106.0, 116.9)
- added H2: MountingHole, kicad-footprints:spacer_m2, F.Cu at (206.6, 59.0)
- added H3: MountingHole, MountingHole:MountingHole_3.5mm_Pad_Via, F.Cu at (95.7, 123.2)
- added H4: MountingHole, MountingHole:MountingHole_3.5mm_Pad_Via, F.Cu at (183.9, 106.3)
- added H5: MountingHole, MountingHole:MountingHole_3.5mm_Pad_Via, F.Cu at (130.4, 46.5)
- added H6: MountingHole, MountingHole:MountingHole_3.5mm_Pad_Via, F.Cu at (139.7, 105.0)
- added H7: MountingHole, MountingHole:MountingHole_3.5mm_Pad_Via, F.Cu at (190.1, 56.8)
- added H8: MountingHole, kicad-footprints:M2_Hole_TH, F.Cu at (81.3, 105.1)
- added H9: MountingHole, kicad-footprints:M2_Hole_TH, F.Cu at (106.3, 90.4)
- added J10: MJ-4PP-9, kicad-footprints:MJ-4PP-9_1side, F.Cu at (77.7, 95.5)
- added J2: USB_C_Receptacle_USB2.0, Connector_USB:USB_C_Receptacle_HRO_TYPE-C-31-M-12, F.Cu at (98.8, 56.4)
- added J4: SWD, Connector_PinHeader_2.54mm:PinHeader_1x04_P2.54mm_Horizontal, F.Cu at (80.4, 63.2)
- added J5: Conn_01x05, Connector_PinHeader_2.54mm:PinHeader_1x05_P2.54mm_Vertical, F.Cu at (137.2, 42.2)
- added J6: Conn_01x03, Connector_PinHeader_2.54mm:PinHeader_1x03_P2.54mm_Vertical, F.Cu at (190.8, 46.6)
- added J7: display, Connector_PinHeader_2.54mm:PinHeader_1x04_P2.54mm_Vertical, F.Cu at (87.5, 88.8)
- added J8: Conn_01x03, Connector_PinHeader_2.54mm:PinHeader_1x03_P2.54mm_Vertical, F.Cu at (114.3, 46.1)
- added J9: MJ-4PP-9, kicad-footprints:MJ-4PP-9_1side, B.Cu at (77.7, 97.3)
- added JP1: SolderJumper_3_Bridged12, Jumper:SolderJumper-3_P1.3mm_Bridged12_Pad1.0x1.5mm, F.Cu at (93.3, 98.6)
- added JP10: SolderJumper_2_Open, kicad-footprints:Jumper, F.Cu at (98.9, 88.2)
- added JP11: SolderJumper_3_Bridged12, Jumper:SolderJumper-3_P1.3mm_Bridged12_Pad1.0x1.5mm, B.Cu at (93.3, 98.6)
- added JP12: SolderJumper_3_Bridged12, Jumper:SolderJumper-3_P1.3mm_Bridged12_Pad1.0x1.5mm, B.Cu at (95.9, 98.6)
- added JP2: SolderJumper_3_Bridged12, Jumper:SolderJumper-3_P1.3mm_Bridged12_Pad1.0x1.5mm, F.Cu at (95.9, 98.6)
- added JP3: SolderJumper_2_Open, kicad-footprints:Jumper, B.Cu at (98.9, 94.1)
- added JP4: SolderJumper_2_Open, kicad-footprints:Jumper, F.Cu at (98.9, 94.1)
- added JP5: SolderJumper_2_Open, kicad-footprints:Jumper, B.Cu at (98.9, 92.1)
- added JP6: SolderJumper_2_Open, kicad-footprints:Jumper, F.Cu at (98.9, 92.1)
- added JP7: SolderJumper_2_Open, kicad-footprints:Jumper, B.Cu at (98.9, 90.2)
- added JP8: SolderJumper_2_Open, kicad-footprints:Jumper, F.Cu at (98.9, 90.2)
- added JP9: SolderJumper_2_Open, kicad-footprints:Jumper, B.Cu at (98.9, 88.2)
- added R10: 22, Resistor_SMD:R_0603_1608Metric_Pad0.98x0.95mm_HandSolder, B.Cu at (101.3, 64.8)
- added R12: 22, Resistor_SMD:R_0603_1608Metric_Pad0.98x0.95mm_HandSolder, B.Cu at (99.6, 64.8)
- added R3: 5.1K, lib:R_0603_1608Metric_Pad0.98x0.95mm_HandSolder, F.Cu at (91.5, 62.8)
- added R9: 22, Resistor_SMD:R_0603_1608Metric_Pad0.98x0.95mm_HandSolder, F.Cu at (101.3, 64.8)
- added SW17: SW_PUSH, lib:MX_ALPS_PG1350_noLed, F.Cu at (197.0, 106.6)
- added SW18: SW_PUSH, lib:MX_ALPS_PG1350_noLed, F.Cu at (216.1, 106.6)
- added SW19: SW_PUSH, lib:MX_ALPS_PG1350_noLed, F.Cu at (101.2, 108.6)
- added SW20: SW_PUSH, lib:MX_ALPS_PG1350_noLed, F.Cu at (80.3, 124.7)
- added SW23: SW_PUSH, lib:MX_ALPS_PG1350_noLed, F.Cu at (130.5, 117.0)
- added SW24: SW_PUSH, lib:MX_ALPS_PG1350_noLed, F.Cu at (151.7, 114.2)
- added SW28: Rotary_Encoder, Rotary_Encoder:RotaryEncoder_Alps_EC11E_Vertical_H20mm, F.Cu at (213.6, 76.0)
- added SW29: Rotary_Encoder, Rotary_Encoder:RotaryEncoder_Alps_EC11E_Vertical_H20mm, F.Cu at (213.6, 114.1)
- added SW30: Rotary_Encoder, Rotary_Encoder:RotaryEncoder_Alps_EC11E_Vertical_H20mm, F.Cu at (168.2, 121.7)
- added SW7: SW_PUSH, lib:MX_ALPS_PG1350_noLed, F.Cu at (120.8, 78.5)
- added U3: holyiot18010, lib:holyiot18010_no_inner, B.Cu at (81.1, 81.2)
- added U4: MX25R3235FM1xx0, Package_SO:SOP-8_3.9x4.9mm_P1.27mm, F.Cu at (109.0, 72.5)
- added U5: TLV73333PDBV, Package_TO_SOT_SMD:SOT-23-5, F.Cu at (109.3, 64.3)
- added U6: TLV73333PDBV, Package_TO_SOT_SMD:SOT-23-5, B.Cu at (109.3, 64.3)
- C1: value C -> 100n; footprint Capacitor_SMD:C_0805_2012Metric_Pad1.18x1.45mm_HandSolder -> Capacitor_SMD:C_0603_1608Metric_Pad1.08x0.95mm_HandSolder; moved to B.Cu
- C2: value C -> 100n; footprint Capacitor_SMD:C_0805_2012Metric_Pad1.18x1.45mm_HandSolder -> Capacitor_SMD:C_0603_1608Metric_Pad1.08x0.95mm_HandSolder
- D1: renamed from D2; footprint Diode_SMD:D_SOD-323_HandSoldering -> lib:D3_SMD_v2_mirror
- D10: renamed from D15; footprint Diode_SMD:D_SOD-323_HandSoldering -> lib:D3_SMD_v2_mirror
- D11: renamed from D19; footprint Diode_SMD:D_SOD-323_HandSoldering -> lib:D3_SMD_v2_mirror
- D12: renamed from D23; footprint Diode_SMD:D_SOD-323_HandSoldering -> lib:D3_SMD_v2_mirror
- D14: renamed from D8; footprint Diode_SMD:D_SOD-323_HandSoldering -> lib:D3_SMD_v2_mirror
- D15: renamed from D12; footprint Diode_SMD:D_SOD-323_HandSoldering -> lib:D3_SMD_v2_mirror
- D16, D4: footprint Diode_SMD:D_SOD-323_HandSoldering -> lib:D3_SMD_v2_mirror
- D17: renamed from D20; footprint Diode_SMD:D_SOD-323_HandSoldering -> lib:D3_SMD_v2_mirror
- D18: renamed from D24; footprint Diode_SMD:D_SOD-323_HandSoldering -> lib:D3_SMD_v2_mirror
- D19: renamed from D5; footprint Diode_SMD:D_SOD-323_HandSoldering -> lib:D3_SMD_v2_mirror
- D2: renamed from D6; footprint Diode_SMD:D_SOD-323_HandSoldering -> lib:D3_SMD_v2_mirror
- D20: renamed from D9; footprint Diode_SMD:D_SOD-323_HandSoldering -> lib:D3_SMD_v2_mirror
- D21: renamed from D13; footprint Diode_SMD:D_SOD-323_HandSoldering -> lib:D3_SMD_v2_mirror
- D22: renamed from D17; footprint Diode_SMD:D_SOD-323_HandSoldering -> lib:D3_SMD_v2_mirror
- D23: renamed from D21; footprint Diode_SMD:D_SOD-323_HandSoldering -> lib:D3_SMD_v2_mirror
- D25: renamed from D1; footprint Diode_SMD:D_SOD-323_HandSoldering -> lib:D3_SMD_v2_mirror
- D3: renamed from D10; footprint Diode_SMD:D_SOD-323_HandSoldering -> lib:D3_SMD_v2_mirror
- D5: renamed from D18; footprint Diode_SMD:D_SOD-323_HandSoldering -> lib:D3_SMD_v2_mirror
- D6: renamed from D22; footprint Diode_SMD:D_SOD-323_HandSoldering -> lib:D3_SMD_v2_mirror
- D7: renamed from D3; footprint Diode_SMD:D_SOD-323_HandSoldering -> lib:D3_SMD_v2_mirror
- D8: renamed from D7; footprint Diode_SMD:D_SOD-323_HandSoldering -> lib:D3_SMD_v2_mirror
- D9: renamed from D11; footprint Diode_SMD:D_SOD-323_HandSoldering -> lib:D3_SMD_v2_mirror
- J3: renamed from J2; moved to B.Cu
- R1, R2: value R -> 4.7K; footprint Resistor_SMD:R_0603_1608Metric_Pad0.98x0.95mm_HandSolder -> lib:R_0603_1608Metric_Pad0.98x0.95mm_HandSolder
- R4: value R -> 5.1K; footprint Resistor_SMD:R_0603_1608Metric_Pad0.98x0.95mm_HandSolder -> lib:R_0603_1608Metric_Pad0.98x0.95mm_HandSolder
- RSW1: footprint kicad-footprints:CherryMX_Choc_Hotswap -> kicad-footprints:ResetSW
- SW1, SW12, SW22, SW6: footprint kicad-footprints:CherryMX_Choc_Hotswap -> lib:MX_ALPS_PG1350_noLed
- SW10: renamed from SW20; footprint kicad-footprints:CherryMX_Choc_Hotswap -> lib:MX_ALPS_PG1350_noLed
- SW11: renamed from SW24; footprint kicad-footprints:CherryMX_Choc_Hotswap -> lib:MX_ALPS_PG1350_noLed
- SW13: renamed from SW7; footprint kicad-footprints:CherryMX_Choc_Hotswap -> lib:MX_ALPS_PG1350_noLed
- SW14: renamed from SW11; footprint kicad-footprints:CherryMX_Choc_Hotswap -> lib:MX_ALPS_PG1350_noLed
- SW15: renamed from SW16; footprint kicad-footprints:CherryMX_Choc_Hotswap -> lib:MX_ALPS_PG1350_noLed
- SW16: renamed from SW21; footprint kicad-footprints:CherryMX_Choc_Hotswap -> lib:MX_ALPS_PG1350_noLed
- SW2: renamed from SW9; footprint kicad-footprints:CherryMX_Choc_Hotswap -> lib:MX_ALPS_PG1350_noLed
- SW21: renamed from SW17; footprint kicad-footprints:CherryMX_Choc_Hotswap -> lib:MX_ALPS_PG1350_noLed
- SW25: renamed from SW4; footprint kicad-footprints:CherryMX_Choc_Hotswap -> lib:MX_ALPS_PG1350_noLed
- SW26: renamed from SW13; footprint kicad-footprints:CherryMX_Choc_Hotswap -> lib:MX_ALPS_reduced
- SW27: renamed from SW18; footprint kicad-footprints:CherryMX_Choc_Hotswap -> lib:MX_ALPS_reduced
- SW3: renamed from SW14; footprint kicad-footprints:CherryMX_Choc_Hotswap -> lib:MX_ALPS_PG1350_noLed
- SW4: renamed from SW19; footprint kicad-footprints:CherryMX_Choc_Hotswap -> lib:MX_ALPS_PG1350_noLed
- SW5: renamed from SW23; footprint kicad-footprints:CherryMX_Choc_Hotswap -> lib:MX_ALPS_PG1350_noLed
- SW8: renamed from SW10; footprint kicad-footprints:CherryMX_Choc_Hotswap -> lib:MX_ALPS_PG1350_noLed
- SW9: renamed from SW15; footprint kicad-footprints:CherryMX_Choc_Hotswap -> lib:MX_ALPS_PG1350_noLed
- U1: value holyiot18010 -> MX25R3235FM1xx0; footprint lib:holyiot18010_mirror -> Package_SO:SOP-8_3.9x4.9mm_P1.27mm; moved to B.Cu
- U2: value M25PX32-VMW -> holyiot18010; footprint Package_SO:SOIJ-8_5.3x5.3mm_P1.27mm -> lib:holyiot18010_no_inner
- moved D12 309.8 mm to (207.5, 86.8), turned to 90 degrees
- moved D6 309.4 mm to (207.5, 66.5), turned to 90 degrees
- moved D5 302.6 mm to (205.6, 66.5), turned to 90 degrees
- moved D17 300.1 mm to (205.6, 106.8), turned to 90 degrees
- moved D18 296.2 mm to (207.5, 106.8), turned to 90 degrees
- moved D11 292.4 mm to (205.6, 86.8), turned to 90 degrees
- moved D9 273.7 mm to (167.5, 70.7), turned to 90 degrees
- moved D3 260.8 mm to (167.5, 53.3), turned to 90 degrees
- moved D4 258.9 mm to (169.4, 53.3), turned to 90 degrees
- moved D16 251.6 mm to (169.4, 89.2), turned to 90 degrees
- moved D10 251.3 mm to (169.4, 70.7), turned to 90 degrees
- moved D15 234.9 mm to (167.5, 89.2), turned to 90 degrees
- moved D2 230.7 mm to (131.3, 59.4), turned to 90 degrees
- moved D23 229.9 mm to (132.1, 125.1), turned to 15 degrees
- moved D8 229.3 mm to (131.3, 76.8), turned to 90 degrees
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- renumbered R3 to R11
Connections:
- net Net-(J2-PadA6) renamed /USBC_+
- net Net-(J2-PadB5) renamed /CC2
- D1 pad 1: /ROW1 -> /ROW0
- D1 pad 2: Net-(D2-Pad2) -> Net-(D1-Pad2)
- D10 pad 1: /ROW2 -> /ROW1
- D10 pad 2: Net-(D15-Pad2) -> Net-(D10-Pad2)
- D11 pad 1: /ROW2 -> /ROW1
- D11 pad 2: Net-(D19-Pad2) (its old number) -> Net-(D11-Pad2)
- D12 pad 1: /ROW2 -> /ROW1
- D12 pad 2: Net-(D23-Pad2) -> Net-(D12-Pad2)
- D14 pad 1: /ROW3 -> /ROW2
- D14 pad 2: Net-(D8-Pad2) -> Net-(D14-Pad2)
- D15 pad 1: /ROW3 -> /ROW2
- D15 pad 2: Net-(D12-Pad2) -> Net-(D15-Pad2)
- D16 pad 1: /ROW3 -> /ROW2
- D17 pad 1: /ROW3 -> /ROW2
- D17 pad 2: Net-(D20-Pad2) -> Net-(D17-Pad2)
- D18 pad 1: /ROW3 -> /ROW2
- D18 pad 2: Net-(D24-Pad2) -> Net-(D18-Pad2)
- D19 pad 1: /ROW0 -> /ROW3
- D2 pad 1: /ROW1 -> /ROW0
- D2 pad 2: Net-(D6-Pad2) -> Net-(D2-Pad2)
- D20 pad 1: /ROW0 -> /ROW3
- D20 pad 2: Net-(D9-Pad2) -> Net-(D20-Pad2)
- D21 pad 1: /ROW0 -> /ROW3
- D21 pad 2: Net-(D13-Pad2) -> Net-(D21-Pad2)
- D22 pad 1: /ROW0 -> /ROW3
- D22 pad 2: Net-(D17-Pad2) -> Net-(D22-Pad2)
- D23 pad 1: /ROW0 -> /ROW3
- D23 pad 2: Net-(D21-Pad2) -> Net-(D23-Pad2)
- D25 pad 1: /ROW0 -> /ROW3
- D25 pad 2: Net-(D1-Pad2) -> Net-(D25-Pad2)
- D3 pad 1: /ROW1 -> /ROW0
- D3 pad 2: Net-(D10-Pad2) -> Net-(D3-Pad2)
- D4 pad 1: /ROW3 -> /ROW0
- D5 pad 1: /ROW1 -> /ROW0
- D5 pad 2: Net-(D18-Pad2) -> Net-(D5-Pad2)
- D6 pad 1: /ROW1 -> /ROW0
- D6 pad 2: Net-(D22-Pad2) -> Net-(D6-Pad2)
- D7 pad 1: /ROW2 -> /ROW1
- D8 pad 1: /ROW2 -> /ROW1
- D8 pad 2: Net-(D7-Pad2) (its old number) -> Net-(D8-Pad2)
- D9 pad 1: /ROW2 -> /ROW1
- D9 pad 2: Net-(D11-Pad2) -> Net-(D9-Pad2)
- J3 pad A5: Net-(J2-PadA5) -> /CC1
- J3 pad A7: Net-(J2-PadA7) -> /USBC_-
- J3 pad A8: Net-(J2-PadA8) -> (no net)
- J3 pad B7: Net-(J2-PadA7) -> /USBC_-
- J3 pad B8: Net-(J2-PadB8) -> (no net)
- R1 pad 1: GND -> /SDA
- R1 pad 2: Net-(J2-PadA5) -> +3V3
- R11 pad 2: /USB+ -> /USBT+
- R2 pad 1: /USB- -> /SCL
- R2 pad 2: Net-(J2-PadA7) -> +3V3
- RSW1 pad 1: /nRESET -> /nReset
- SW10 pad 1: /COL4 -> /COL3
- SW10 pad 2: Net-(D20-Pad2) -> Net-(D10-Pad2)
- SW11 pad 1: /COL5 -> /COL4
- SW11 pad 2: Net-(D24-Pad2) -> Net-(D11-Pad2)
- SW12 pad 1: /COL2 -> /COL5
- SW13 pad 1: /COL1 -> /COL0
- SW13 pad 2: Net-(D7-Pad2) (its old number) -> Net-(D13-Pad2)
- SW14 pad 1: /COL2 -> /COL1
- SW14 pad 2: Net-(D11-Pad2) -> Net-(D14-Pad2)
- SW15 pad 1: /COL3 -> /COL2
- SW15 pad 2: Net-(D16-Pad2) -> Net-(D15-Pad2)
- SW16 pad 1: /COL5 -> /COL3
- SW16 pad 2: Net-(D21-Pad2) -> Net-(D16-Pad2)
- SW2 pad 1: /COL2 -> /COL1
- SW2 pad 2: Net-(D9-Pad2) -> Net-(D2-Pad2)
- SW21 pad 1: /COL4 -> /COL6
- SW21 pad 2: Net-(D17-Pad2) -> Net-(D21-Pad2)
- SW22 pad 1: /COL5 -> /COL2
- SW25 pad 1: /COL0 -> /COL5
- SW25 pad 2: Net-(D4-Pad2) -> Net-(D25-Pad2)
- SW26 pad 1: /COL3 -> /COL6
- SW26 pad 2: Net-(D13-Pad2) -> Net-(D21-Pad2)
- SW27 pad 1: /COL4 -> /COL2
- SW27 pad 2: Net-(D18-Pad2) -> /ROW3
- SW3 pad 1: /COL3 -> /COL2
- SW3 pad 2: Net-(D14-Pad2) -> Net-(D3-Pad2)
- SW4 pad 1: /COL4 -> /COL3
- SW4 pad 2: Net-(D19-Pad2) (its old number) -> Net-(D4-Pad2)
- SW5 pad 1: /COL5 -> /COL4
- SW5 pad 2: Net-(D23-Pad2) -> Net-(D5-Pad2)
- SW6 pad 1: /COL1 -> /COL5
- SW8 pad 1: /COL2 -> /COL1
- SW8 pad 2: Net-(D10-Pad2) -> Net-(D8-Pad2)
- SW9 pad 1: /COL3 -> /COL2
- SW9 pad 2: Net-(D15-Pad2) -> Net-(D9-Pad2)
- U1 pad 1: GND -> /nCS_B
- U1 pad 2: Net-(U1-Pad2) -> /SIO1_B
- U1 pad 3: Net-(U1-Pad3) -> /SIO2_B
- U1 pad 4: Net-(U1-Pad4) -> GND
- U1 pad 5: Net-(U1-Pad5) -> /SIO0_B
- U1 pad 6: Net-(U1-Pad6) -> /SCLK_B
- U1 pad 7: Net-(U1-Pad7) -> /SIO3_B
- U1 pad 8: Net-(U1-Pad8) -> +3V3
- U2 pad 1: Net-(U2-Pad1) -> GND
- U2 pad 2: Net-(U2-Pad2) -> /COL0
- U2 pad 3: Net-(U2-Pad3) -> /COL1
- U2 pad 4: GND -> (no net)
- U2 pad 5: Net-(U2-Pad5) -> (no net)
- U2 pad 6: Net-(U2-Pad6) -> /ROW1
- U2 pad 7: Net-(U2-Pad7) -> /ROW0
- U2 pad 8: +3V3 -> /ROW2
Routing:
- net /COL5: track 0.00 -> 305.4 mm, vias 0 -> 7
- net /COL4: track 0.00 -> 270.7 mm, vias 0 -> 5
- net /QDEC_B: track 0.00 -> 269.3 mm, vias 0 -> 3
- net /COL3: track 0.00 -> 268.5 mm, vias 0 -> 9
- net /ROW3: track 0.00 -> 265.9 mm, vias 0 -> 9
- net /QDEC_A: track 0.00 -> 265.3 mm, vias 0 -> 3
- net /ROW2: track 0.00 -> 263.7 mm, vias 0 -> 9
- net /COL2: track 42.7 -> 279.8 mm, vias 1 -> 10
- net /COL1: track 0.00 -> 227.1 mm, vias 0 -> 8
- net /ROW1: track 0.00 -> 220.2 mm, vias 0 -> 7
- net /ROW0: track 0.00 -> 212.7 mm, vias 0 -> 7
- net /COL6: track 0.00 -> 195.5 mm, vias 0 -> 3
- net /COL0: track 46.8 -> 211.8 mm, vias 0 -> 8
- net +3V3: track 0.00 -> 134.0 mm, vias 0 -> 7
- net /UART0_RX: track 0.00 -> 105.5 mm, vias 0 -> 4
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- added copper zone on B.Cu, net GND
- added copper zone on F.Cu, net GND
Other:
- outline, holes or cut-outs redrawn
- net class Default: clearance 0.2 -> 0.2032
- rule pad_to_mask_clearance: 0 -> 0.05
- rule trace_clearance: 0.2 -> 0.2032
- rule trace_min: 0.2 -> 0.2032
- rule via_min_drill: 0.3 -> 0.2
- board text added: "Type C"

Commit message: Update to latest design
Parts:
- removed D14, D15, D16, D17, D18, D19, D20, D21, D22, D23, D24, D25: D, lib:D3_SMD_v2_mirror
- added J1: Conn_02x05_Odd_Even, Connector_PinHeader_1.27mm:PinHeader_2x05_P1.27mm_Vertical_SMD, F.Cu at (87.1, 52.0)
- D1, D10, D11, D13, D2, D3, D4, D5, D6, D7, D8, D9: value D -> BAS40-05; footprint lib:D3_SMD_v2_mirror -> lib:SOT-23_mirror; moved to B.Cu
- D12: value D -> BAS40-05; footprint lib:D3_SMD_v2_mirror -> lib:SOT-23_mirror
- J4: value SWD -> Conn_02x05_Odd_Even; footprint Connector_PinHeader_2.54mm:PinHeader_1x04_P2.54mm_Horizontal -> Connector_PinHeader_1.27mm:PinHeader_2x05_P1.27mm_Vertical_SMD; moved to B.Cu
- U1, U4: value MX25R3235FM1xx0 -> BY25Q32BSTIG(T)
- moved D11 114.4 mm to (92.8, 105.9), turned to 225 degrees
- moved D10 85.6 mm to (90.3, 103.3), turned to 45 degrees
- moved D12 66.5 mm to (143.4, 104.3), turned to 0 degrees
- moved D9 47.9 mm to (208.8, 95.0), turned to 0 degrees
- moved D2 43.5 mm to (170.7, 40.8), turned to 0 degrees
- moved D3 41.4 mm to (208.8, 56.8), turned to 0 degrees
- moved D8 39.4 mm to (170.7, 79.4), turned to 0 degrees
- moved D4 38.6 mm to (132.6, 64.7), turned to 0 degrees
- moved D5 35.4 mm to (170.6, 61.1), turned to 0 degrees
- moved D13 34.9 mm to (163.4, 102.5), turned to 0 degrees
- moved J4 13.0 mm to (87.1, 52.0), turned to 180 degrees
- moved D6 10.4 mm to (208.8, 76.8), turned to 0 degrees
- moved D1 8.93 mm to (132.6, 51.0), turned to 0 degrees
- moved J10 8.85 mm to (80.2, 87.1)
- moved J9 8.85 mm to (80.2, 88.8)
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Connections:
- D1 pad 1: /ROW0 -> Net-(D1-Pad1)
- D10 pad 1: /ROW1 -> Net-(D10-Pad1)
- D11 pad 1: /ROW1 -> Net-(D11-Pad1)
- D12 pad 1: /ROW1 -> /ROW3
- D13 pad 1: /ROW2 -> Net-(D13-Pad1)
- D2 pad 1: /ROW0 -> Net-(D2-Pad1)
- D3 pad 1: /ROW0 -> Net-(D3-Pad1)
- D4 pad 1: /ROW0 -> Net-(D4-Pad1)
- D5 pad 1: /ROW0 -> Net-(D5-Pad1)
- D6 pad 1: /ROW0 -> Net-(D6-Pad1)
- D7 pad 1: /ROW1 -> Net-(D7-Pad1)
- D8 pad 1: /ROW1 -> Net-(D8-Pad1)
- D9 pad 1: /ROW1 -> Net-(D9-Pad1)
- J10 pad A: GND -> +3V3
- J10 pad B: +3V3 -> GND
- J4 pad 3: /SWCLK -> GND
- J4 pad 4: GND -> /SWCLK
- J9 pad A: GND -> +3V3
- J9 pad B: +3V3 -> GND
- SW1 pad 2: Net-(D1-Pad2) -> Net-(D1-Pad1)
- SW10 pad 2: Net-(D10-Pad2) -> Net-(D5-Pad2)
- SW11 pad 2: Net-(D11-Pad2) -> Net-(D6-Pad1)
- SW12 pad 2: Net-(D12-Pad2) -> Net-(D6-Pad2)
- SW13 pad 2: Net-(D13-Pad2) -> Net-(D7-Pad1)
- SW14 pad 2: Net-(D14-Pad2) -> Net-(D7-Pad2)
- SW15 pad 2: Net-(D15-Pad2) -> Net-(D8-Pad1)
- SW16 pad 2: Net-(D16-Pad2) -> Net-(D8-Pad2)
- SW17 pad 2: Net-(D17-Pad2) -> Net-(D9-Pad1)
- SW18 pad 2: Net-(D18-Pad2) -> Net-(D9-Pad2)
- SW19 pad 2: Net-(D19-Pad2) -> Net-(D11-Pad1)
- SW2 pad 2: Net-(D2-Pad2) -> Net-(D1-Pad2)
- SW20 pad 2: Net-(D20-Pad2) -> Net-(D10-Pad2)
- SW21 pad 2: Net-(D21-Pad2) -> Net-(D10-Pad1)
- SW22 pad 2: Net-(D22-Pad2) -> Net-(D11-Pad2)
- SW23 pad 2: Net-(D23-Pad2) -> Net-(D12-Pad2)
- SW24 pad 2: Net-(D24-Pad2) -> Net-(D13-Pad1)
- SW25 pad 2: Net-(D25-Pad2) -> Net-(D13-Pad2)
- SW26 pad 2: Net-(D21-Pad2) -> Net-(D10-Pad1)
- SW27 pad 2: /ROW3 -> Net-(D11-Pad2)
- SW3 pad 2: Net-(D3-Pad2) -> Net-(D2-Pad1)
- SW4 pad 2: Net-(D4-Pad2) -> Net-(D2-Pad2)
- SW5 pad 2: Net-(D5-Pad2) -> Net-(D3-Pad1)
- SW6 pad 2: Net-(D6-Pad2) -> Net-(D3-Pad2)
- SW7 pad 2: Net-(D7-Pad2) -> Net-(D4-Pad1)
- SW8 pad 2: Net-(D8-Pad2) -> Net-(D4-Pad2)
- SW9 pad 2: Net-(D9-Pad2) -> Net-(D5-Pad1)
- U2 pad 5: (no net) -> /ROW1
- U2 pad 6: /ROW1 -> /CC1
- U3 pad 36: (no net) -> GND
- U3 pad 5: (no net) -> /ROW1
- U3 pad 6: /ROW1 -> /CC1
Routing:
- net Net-(D10-Pad1): track 0.00 -> 65.9 mm, vias 0 -> 4
- net Net-(D21-Pad2): track 44.1 -> 0.00 mm, vias 2 -> 0
- net /nReset: track 28.1 -> 63.6 mm, vias 2 -> 4
- net /ROW3: track 265.9 -> 237.1 mm, vias 9 -> 8
- net Net-(D11-Pad2): track 13.6 -> 41.6 mm, vias 1 -> 2
- net Net-(D19-Pad2): track 25.9 -> 0.00 mm, vias 1 -> 0
- net /CC1: track 12.1 -> 36.7 mm, vias 3 -> 5
- net Net-(D25-Pad2): track 24.2 -> 0.00 mm, vias 2 -> 0
- net Net-(D18-Pad2): track 24.2 -> 0.00 mm, vias 2 -> 0
- net Net-(D11-Pad1): track 0.00 -> 23.3 mm, vias 0 -> 1
- net Net-(D23-Pad2): track 20.1 -> 0.00 mm, vias 1 -> 0
- net Net-(D14-Pad2): track 19.4 -> 0.00 mm, vias 1 -> 0
- net Net-(D20-Pad2): track 18.0 -> 0.00 mm, vias 1 -> 0
- net Net-(D16-Pad2): track 16.2 -> 0.00 mm, vias 1 -> 0
- net +3V3: track 134.0 -> 118.3 mm, vias 7 -> 8
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Other:
- outline, holes or cut-outs redrawn
- board text added: "1"
- board text added: "COL6"
- board text added: "GND"
- board text added: "JLCJLCJLCJLC"
- board text added: "Noria v0.1"
- board text added: "QA"
- board text added: "QB"
- board text added: "ROW0"
- board text added: "ROW1"
- board text added: "ROW2"
- board text added: "ROW3"
- board text added: "RX"
- board text added: "TX"

Commit message: And another update
Other:
- net class Default removed
